Commit message: Modify the height of the robot

File: include/urdf/wild_thumper.urdf.xacro (robot description, xacro)
@@ -39,5 +39,5 @@
                         <origin xyz="0 0 0" rpy="0 0 0"/>
 			<geometry>
-				<box size="0.24 0.12 0.01"/>
+				<box size="0.24 0.12 0.03"/>
 			</geometry>
 		</visual>
@@ -68,17 +68,17 @@
 	</joint>
         <joint name="mount_spacer_joint" type="fixed">
-		<parent link="base_footprint"/>
+		<parent link="base_link"/>
 		<child link="mount_spacers"/>
-		<origin xyz="-0.005 0.0 0.132" rpy="0 0 0"/>
+		<origin xyz="0.00 0.0 0.06" rpy="0 0 0"/>
 	</joint>
         <joint name="mount_lidar" type="fixed">
 		<parent link="base_link"/>
 		<child link="mount_lidar"/>
-		<origin xyz="-0.07 0 0.066" rpy="0 0 0"/>
+		<origin xyz="-0.07 0 0.086" rpy="0 0 0"/>
 	</joint>
        <joint name="laser" type="fixed">
 		<parent link="base_link"/>
 		<child link="laser"/>
-                <origin xyz="-0.08 0 0.130" rpy="0 0 0"/>
+                <origin xyz="-0.08 0 0.150" rpy="0 0 0"/>
 	</joint>
         <xacro:macro name="wheel" params="pos side xyz rpy">
@@ -119,5 +119,5 @@
             </link>
             <joint name="${sensor}_${num}_spacer_joint" type="continuous">
-		<parent link="base_link"/>
+		<parent link="mount_spacers"/>
 		<child link="${sensor}_${num}_spacer"/>
 		<origin xyz="${xyz}" rpy="0 0 0"/>
@@ -128,11 +128,11 @@
 	<xacro:wheel pos="front" side="left"  xyz=" 0.07525  0.12 -0.025" rpy="0 0 0" />
 	<xacro:wheel pos="front" side="right" xyz=" 0.07525 -0.12 -0.025" rpy="0 0 0" />
-        <xacro:spacer sensor="lidar" num="1_1" len="0.01" rad="0.0025" xyz="-0.03 -0.04 0.060" />
-        <xacro:spacer sensor="lidar" num="1_2" len="0.01" rad="0.0025" xyz="-0.03  0.04 0.060" />
-        <xacro:spacer sensor="lidar" num="1_3" len="0.01" rad="0.0025" xyz="-0.11 -0.04 0.060" />
-        <xacro:spacer sensor="lidar" num="1_4" len="0.01" rad="0.0025" xyz="-0.11  0.04 0.060" />
-        <xacro:spacer sensor="lidar" num="2_1" len="0.02" rad="0.0028" xyz="-0.035 -0.02 0.075" />
-        <xacro:spacer sensor="lidar" num="2_2" len="0.02" rad="0.0028" xyz="-0.035  0.02 0.075" />
-        <xacro:spacer sensor="lidar" num="2_3" len="0.02" rad="0.0028" xyz="-0.105 -0.028 0.075" />
-        <xacro:spacer sensor="lidar" num="2_4" len="0.02" rad="0.0028" xyz="-0.105  0.028 0.075" />
+        <xacro:spacer sensor="lidar" num="1_1" len="0.01" rad="0.0025" xyz="-0.03 -0.04 0.020" />
+        <xacro:spacer sensor="lidar" num="1_2" len="0.01" rad="0.0025" xyz="-0.03  0.04 0.020" />
+        <xacro:spacer sensor="lidar" num="1_3" len="0.01" rad="0.0025" xyz="-0.11 -0.04 0.020" />
+        <xacro:spacer sensor="lidar" num="1_4" len="0.01" rad="0.0025" xyz="-0.11  0.04 0.020" />
+        <xacro:spacer sensor="lidar" num="2_1" len="0.02" rad="0.0028" xyz="-0.035 -0.02 0.035" />
+        <xacro:spacer sensor="lidar" num="2_2" len="0.02" rad="0.0028" xyz="-0.035  0.02 0.035" />
+        <xacro:spacer sensor="lidar" num="2_3" len="0.02" rad="0.0028" xyz="-0.105 -0.028 0.035" />
+        <xacro:spacer sensor="lidar" num="2_4" len="0.02" rad="0.0028" xyz="-0.105  0.028 0.035" />
 </robot>

Commit message: Fix urdf working with laser

File: include/urdf/wild_thumper.urdf.xacro (robot description, xacro)
@@ -5,14 +5,4 @@
            <color rgba="${45/255} ${45/255} ${45/255} 1.0"/>
         </material>
-	<link name="base_footprint">
-		<visual>
-			<geometry>
-				<box size="0.28 0.31 0.000001"/>
-			</geometry>
-			<material name="grey">
-				<color rgba="0.5 0.5 0.5 0.5"/>
-			</material>
-		</visual>
-	</link>
 	<link name="base_link">
 		<collision>
@@ -28,9 +18,4 @@
 			</geometry>
 		</visual>
-		<inertial>
-			<origin xyz="-0.00275 0 -0.02" rpy="0 0 0"/>
-			<mass value="2.5"/>
-			<inertia ixx="0.012708" ixy="0.0" ixz="0.0" iyy="0.0084375" iyz="0.0" izz="0.017771"/>
-		</inertial>
 	</link>
         <link name="mount_spacers">
@@ -62,9 +47,4 @@
 		</visual>
 	</link>
-	<joint name="base_link_joint" type="fixed">
-		<parent link="base_footprint"/>
-		<child link="base_link"/>
-		<origin xyz="0.0 0.0 0.082" rpy="0 0 0"/>
-	</joint>
         <joint name="mount_spacer_joint" type="fixed">
 		<parent link="base_link"/>

Commit message: Add basefootprint to urdf

File: include/urdf/wild_thumper.urdf.xacro (robot description, xacro)
@@ -5,4 +5,14 @@
            <color rgba="${45/255} ${45/255} ${45/255} 1.0"/>
         </material>
+        <link name="base_footprint">
+		<visual>
+			<geometry>
+				<box size="0.28 0.31 0.000001"/>
+			</geometry>
+			<material name="grey">
+				<color rgba="0.5 0.5 0.5 0.5"/>
+			</material>
+		</visual>
+	</link>
 	<link name="base_link">
 		<collision>
@@ -18,4 +28,9 @@
 			</geometry>
 		</visual>
+                <inertial>
+			<origin xyz="-0.00275 0 -0.02" rpy="0 0 0"/>
+			<mass value="2.5"/>
+			<inertia ixx="0.012708" ixy="0.0" ixz="0.0" iyy="0.0084375" iyz="0.0" izz="0.017771"/>
+		</inertial>
 	</link>
         <link name="mount_spacers">
@@ -47,4 +62,9 @@
 		</visual>
 	</link>
+        <joint name="base_link_joint" type="fixed">
+		<parent link="base_footprint"/>
+		<child link="base_link"/>
+		<origin xyz="0.0 0.0 0.082" rpy="0 0 0"/>
+	</joint>
         <joint name="mount_spacer_joint" type="fixed">
 		<parent link="base_link"/>

Commit message: Changes to URDF to test odom

File: include/urdf/wild_thumper.urdf.xacro (robot description, xacro)
@@ -5,14 +5,4 @@
            <color rgba="${45/255} ${45/255} ${45/255} 1.0"/>
         </material>
-        <link name="base_footprint">
-		<visual>
-			<geometry>
-				<box size="0.28 0.31 0.000001"/>
-			</geometry>
-			<material name="grey">
-				<color rgba="0.5 0.5 0.5 0.5"/>
-			</material>
-		</visual>
-	</link>
 	<link name="base_link">
 		<collision>
@@ -28,10 +18,5 @@
 			</geometry>
 		</visual>
-                <inertial>
-			<origin xyz="-0.00275 0 -0.02" rpy="0 0 0"/>
-			<mass value="2.5"/>
-			<inertia ixx="0.012708" ixy="0.0" ixz="0.0" iyy="0.0084375" iyz="0.0" izz="0.017771"/>
-		</inertial>
-	</link>
+       </link>
         <link name="mount_spacers">
 		<visual>
@@ -62,9 +47,4 @@
 		</visual>
 	</link>
-        <joint name="base_link_joint" type="fixed">
-		<parent link="base_footprint"/>
-		<child link="base_link"/>
-		<origin xyz="0.0 0.0 0.082" rpy="0 0 0"/>
-	</joint>
         <joint name="mount_spacer_joint" type="fixed">
 		<parent link="base_link"/>

Commit message: Fixing odometry msgs

File: include/urdf/wild_thumper.urdf.xacro (robot description, xacro)
@@ -3,6 +3,13 @@
 	<xacro:property name="PI" value="3.1415926535897931" />
         <material name="Black">
-           <color rgba="${45/255} ${45/255} ${45/255} 1.0"/>
+            <color rgba="${45/255} ${45/255} ${45/255} 1.0"/>
         </material>
+        <link name="base_footprint">
+            <visual>
+                <geometry>
+                    <box size="0.28 0.31 0.000001"/>
+                </geometry>
+            </visual>
+        </link>
 	<link name="base_link">
 		<collision>
@@ -13,5 +20,5 @@
 		<visual>
                         <material name="Black"/>
-                        <origin xyz="-0.00275 0 0" rpy="0 0 0"/>
+                        <origin xyz="-0.00275 0 0.0" rpy="0 0 0"/>
 			<geometry>
 				<mesh filename="package://wild_thumper/include/meshes/wild_thumper_4wd.stl" />
@@ -47,4 +54,9 @@
 		</visual>
 	</link>
+        <joint name="base_link_joint" type="fixed">
+                <origin rpy="0 0 0" xyz="0 0 -0.082 "/>
+                <child link="base_footprint"/>
+                <parent link="base_link"/>
+        </joint>
         <joint name="mount_spacer_joint" type="fixed">
 		<parent link="base_link"/>

Commit message: Add imu to the urdf file

File: include/urdf/wild_thumper.urdf.xacro (robot description, xacro)
@@ -35,5 +35,5 @@
 		</visual>
 	</link>
-        <link name="mount_lidar">
+    <link name="mount_lidar">
 		<visual>
                         <material name="Black"/>
@@ -44,5 +44,5 @@
 		</visual>
 	</link>
-        <link name="laser">
+    <link name="laser">
 		<visual>
                         <material name="Black"/>
@@ -54,23 +54,35 @@
 		</visual>
 	</link>
-        <joint name="base_link_joint" type="fixed">
-                <origin rpy="0 0 0" xyz="0 0 -0.082 "/>
-                <child link="base_footprint"/>
-                <parent link="base_link"/>
-        </joint>
-        <joint name="mount_spacer_joint" type="fixed">
+	<link name="imu_link">
+		<visual>
+                <geometry>
+                    <box size="0.02 0.02 0.02"/>
+                </geometry>
+            </visual>
+	</link>
+    <joint name="base_link_joint" type="fixed">
+        <origin rpy="0 0 0" xyz="0 0 -0.082 "/>
+        <child link="base_footprint"/>
+        <parent link="base_link"/>
+    </joint>
+    <joint name="mount_spacer_joint" type="fixed">
 		<parent link="base_link"/>
 		<child link="mount_spacers"/>
 		<origin xyz="0.00 0.0 0.06" rpy="0 0 0"/>
 	</joint>
-        <joint name="mount_lidar" type="fixed">
+    <joint name="mount_lidar" type="fixed">
 		<parent link="base_link"/>
 		<child link="mount_lidar"/>
 		<origin xyz="-0.07 0 0.086" rpy="0 0 0"/>
 	</joint>
-       <joint name="laser" type="fixed">
+    <joint name="laser" type="fixed">
 		<parent link="base_link"/>
 		<child link="laser"/>
-                <origin xyz="-0.08 0 0.150" rpy="0 0 0"/>
+        <origin xyz="-0.08 0 0.150" rpy="0 0 0"/>
+	</joint>
+    <joint name="base_imu_link" type="fixed">
+		<parent link="base_link"/>
+		<child link="imu_link"/>
+        <origin xyz="0.00 0 0.10" rpy="0 0 0"/>
 	</joint>
         <xacro:macro name="wheel" params="pos side xyz rpy">

Commit message: Update name of link and joint of the imu in the urdf file

File: include/urdf/wild_thumper.urdf.xacro (robot description, xacro)
@@ -54,5 +54,5 @@
 		</visual>
 	</link>
-	<link name="imu_link">
+	<link name="base_imu_link">
 		<visual>
                 <geometry>
@@ -81,7 +81,7 @@
         <origin xyz="-0.08 0 0.150" rpy="0 0 0"/>
 	</joint>
-    <joint name="base_imu_link" type="fixed">
+    <joint name="base_imu" type="fixed">
 		<parent link="base_link"/>
-		<child link="imu_link"/>
+		<child link="base_imu_link"/>
         <origin xyz="0.00 0 0.10" rpy="0 0 0"/>
 	</joint>

Commit message: Update position of the imu in the urdf

File: include/urdf/wild_thumper.urdf.xacro (robot description, xacro)
@@ -84,10 +84,10 @@
 		<parent link="base_link"/>
 		<child link="base_imu_link"/>
-        <origin xyz="0.00 0 0.10" rpy="0 0 0"/>
+        <origin xyz="0.05 -0.01 0.09" rpy="0 0 0"/>
 	</joint>
-        <xacro:macro name="wheel" params="pos side xyz rpy">
+    <xacro:macro name="wheel" params="pos side xyz rpy">
 		<link name="${pos}_${side}_wheel">
 			<visual>
-                                <material name="Black"/>
+                <material name="Black"/>
 				<origin xyz="0 0 0" rpy="0 0 0"/>
 				<geometry>
@@ -104,5 +104,5 @@
 				<origin xyz="0 0 0" rpy="0 0 0"/>
 				<mass value="0.2"/>
-				<inertia ixx="0.00024" ixy="0" ixz="0" iyy="0.00036" iyz="0" izz="0.00024"/>
+				<inertia ixx="0.00024" ixy="0" ixz="0" iyy="0.00024" iyz="0" izz="0.00024"/>
 			</inertial>
 		</link>
@@ -114,5 +114,5 @@
 		</joint>
 	</xacro:macro>
-        <xacro:macro name="spacer" params="sensor num len rad xyz">
+    <xacro:macro name="spacer" params="sensor num len rad xyz">
              <link name="${sensor}_${num}_spacer">
                 <visual>
@@ -127,16 +127,16 @@
 		<origin xyz="${xyz}" rpy="0 0 0"/>
             </joint>
-        </xacro:macro>
-        <xacro:wheel pos="rear" side="left"   xyz="-0.07525  0.12 -0.025" rpy="0 0 0" />
-	<xacro:wheel pos="rear" side="right"  xyz="-0.07525 -0.12 -0.025" rpy="0 0 0" />
-	<xacro:wheel pos="front" side="left"  xyz=" 0.07525  0.12 -0.025" rpy="0 0 0" />
-	<xacro:wheel pos="front" side="right" xyz=" 0.07525 -0.12 -0.025" rpy="0 0 0" />
-        <xacro:spacer sensor="lidar" num="1_1" len="0.01" rad="0.0025" xyz="-0.03 -0.04 0.020" />
-        <xacro:spacer sensor="lidar" num="1_2" len="0.01" rad="0.0025" xyz="-0.03  0.04 0.020" />
-        <xacro:spacer sensor="lidar" num="1_3" len="0.01" rad="0.0025" xyz="-0.11 -0.04 0.020" />
-        <xacro:spacer sensor="lidar" num="1_4" len="0.01" rad="0.0025" xyz="-0.11  0.04 0.020" />
-        <xacro:spacer sensor="lidar" num="2_1" len="0.02" rad="0.0028" xyz="-0.035 -0.02 0.035" />
-        <xacro:spacer sensor="lidar" num="2_2" len="0.02" rad="0.0028" xyz="-0.035  0.02 0.035" />
-        <xacro:spacer sensor="lidar" num="2_3" len="0.02" rad="0.0028" xyz="-0.105 -0.028 0.035" />
-        <xacro:spacer sensor="lidar" num="2_4" len="0.02" rad="0.0028" xyz="-0.105  0.028 0.035" />
+    </xacro:macro>
+    <xacro:wheel pos="rear" side="left"  xyz="-0.07525 0.12 -0.025" rpy="0 0 0" />
+    <xacro:wheel pos="rear" side="right"  xyz="-0.07525 -0.12 -0.025" rpy="0 0 0" />
+	<xacro:wheel pos="front" side="left"  xyz="0.07525 0.12 -0.025" rpy="0 0 0" />
+	<xacro:wheel pos="front" side="right" xyz="0.07525 -0.12 -0.025" rpy="0 0 0" />
+    <xacro:spacer sensor="lidar" num="1_1" len="0.01" rad="0.0025" xyz="-0.03 -0.04 0.020" />
+    <xacro:spacer sensor="lidar" num="1_2" len="0.01" rad="0.0025" xyz="-0.03 0.04 0.020" />
+    <xacro:spacer sensor="lidar" num="1_3" len="0.01" rad="0.0025" xyz="-0.11 -0.04 0.020" />
+    <xacro:spacer sensor="lidar" num="1_4" len="0.01" rad="0.0025" xyz="-0.11 0.04 0.020" />
+    <xacro:spacer sensor="lidar" num="2_1" len="0.02" rad="0.0028" xyz="-0.035 -0.02 0.035" />
+    <xacro:spacer sensor="lidar" num="2_2" len="0.02" rad="0.0028" xyz="-0.035 0.02 0.035" />
+    <xacro:spacer sensor="lidar" num="2_3" len="0.02" rad="0.0028" xyz="-0.105 -0.028 0.035" />
+    <xacro:spacer sensor="lidar" num="2_4" len="0.02" rad="0.0028" xyz="-0.105 0.028 0.035" />
 </robot>

Commit message: Changed base_footprint to be the parent node

File: include/urdf/wild_thumper.urdf.xacro (robot description, xacro)
@@ -62,7 +62,7 @@
 	</link>
     <joint name="base_link_joint" type="fixed">
-        <origin rpy="0 0 0" xyz="0 0 -0.082 "/>
-        <child link="base_footprint"/>
-        <parent link="base_link"/>
+        <origin rpy="0 0 0" xyz="0 0 0.082 "/>
+        <child link="base_link"/>
+        <parent link="base_footprint"/>
     </joint>
     <joint name="mount_spacer_joint" type="fixed">

Commit message: Change odom child in the odometry node

File: include/urdf/wild_thumper.urdf.xacro (robot description, xacro)
@@ -5,5 +5,5 @@
             <color rgba="${45/255} ${45/255} ${45/255} 1.0"/>
         </material>
-        <link name="base_footprint">
+    <link name="base_footprint">
             <visual>
                 <geometry>

Commit message: Align code in the urdf

File: include/urdf/wild_thumper.urdf.xacro (robot description, xacro)
@@ -19,6 +19,6 @@
 		</collision>
 		<visual>
-                        <material name="Black"/>
-                        <origin xyz="-0.00275 0 0.0" rpy="0 0 0"/>
+            <material name="Black"/>
+            <origin xyz="-0.00275 0 0.0" rpy="0 0 0"/>
 			<geometry>
 				<mesh filename="package://wild_thumper/include/meshes/wild_thumper_4wd.stl" />
@@ -28,8 +28,8 @@
         <link name="mount_spacers">
 		<visual>
-                        <material name="Black"/>
-                        <origin xyz="0 0 0" rpy="0 0 0"/>
+            <material name="Black"/>
+            <origin xyz="0 0 0" rpy="0 0 0"/>
 			<geometry>
-				<box size="0.24 0.12 0.03"/>
+			<box size="0.24 0.12 0.03"/>
 			</geometry>
 		</visual>
@@ -37,6 +37,6 @@
     <link name="mount_lidar">
 		<visual>
-                        <material name="Black"/>
-                        <origin xyz="0 0 0" rpy="0 0 0"/>
+            <material name="Black"/>
+            <origin xyz="0 0 0" rpy="0 0 0"/>
 			<geometry>
 				<box size="0.09 0.087 0.002"/>
@@ -46,8 +46,8 @@
     <link name="laser">
 		<visual>
-                        <material name="Black"/>
-                        <axis xyz="1 0 0" rpy="0 0 0"/>
-                        <origin xyz="-0.032 0.035 -0.045" rpy="${PI/2} 0 0"/>
-               		<geometry>
+            <material name="Black"/>
+            <axis xyz="1 0 0" rpy="0 0 0"/>
+            <origin xyz="-0.032 0.035 -0.045" rpy="${PI/2} 0 0"/>
+            <geometry>
 				<mesh filename="package://wild_thumper/include/meshes/rplidar.stl" scale="0.001 0.001 0.001"/>
 			</geometry>
@@ -56,13 +56,13 @@
 	<link name="base_imu_link">
 		<visual>
-                <geometry>
-                    <box size="0.02 0.02 0.02"/>
-                </geometry>
-            </visual>
+            <geometry>
+                <box size="0.02 0.02 0.02"/>
+            </geometry>
+        </visual>
 	</link>
     <joint name="base_link_joint" type="fixed">
+	    <parent link="base_footprint"/>
+	    <child link="base_link"/>
         <origin rpy="0 0 0" xyz="0 0 0.082 "/>
-        <child link="base_link"/>
-        <parent link="base_footprint"/>
     </joint>
     <joint name="mount_spacer_joint" type="fixed">

Commit message: Add razor imu to the urdf

File: include/urdf/wild_thumper.urdf.xacro (robot description, xacro)
@@ -11,5 +11,6 @@
                 </geometry>
             </visual>
-        </link>
+    </link>
+	*
 	<link name="base_link">
 		<collision>
@@ -25,6 +26,6 @@
 			</geometry>
 		</visual>
-       </link>
-        <link name="mount_spacers">
+    </link>
+    <link name="mount_spacers">
 		<visual>
             <material name="Black"/>
